File: cartridge_controller.sch (KiCad schematic (older format))
At the start: 20 parts, among them J9 Micro_SD_Card_Det, U13 STM32F407VGTx

Commit message: C64 Emulation. First run on my beloved ATARI 130XE.
Parts:
- C10, C11, C12, C13, C14, C15, C6, C7, C8, C9: footprint Capacitors_SMD:C_1206_HandSoldering -> Capacitor_SMD:C_1206_3216Metric_Pad1.42x1.75mm_HandSolder; symbol C_Small -> Device1:C_Small
- D3, D4: footprint LEDs:LED_1206 -> LED_SMD:LED_1206_3216Metric_Pad1.42x1.75mm_HandSolder; symbol Led_Small -> atari23MTS_Upgrade-rescue:Led_Small
- J9: symbol Micro_SD_Card_Det -> Connector1:Micro_SD_Card_Det
- R5, R6, R7, R8, R9: footprint Resistors_SMD:R_1206_HandSoldering -> Resistor_SMD:R_1206_3216Metric_Pad1.42x1.75mm_HandSolder; symbol R_Small -> Device1:R_Small
- U13: footprint Housings_QFP:TQFP-100_14x14mm_Pitch0.5mm -> Package_QFP:TQFP-100-1EP_14x14mm_P0.5mm_EP5x5mm; symbol STM32F407VGTx -> MCU_ST_STM32F41:STM32F407VGTx
- XT1: symbol Crystal_Small -> Device1:Crystal_Small
