File: memory_controller.sch (KiCad schematic (older format))
At the start: 19 parts, among them U14 STM32F407VGTx

Commit message: C64 Emulation. First run on my beloved ATARI 130XE.
Parts:
- C16, C17, C18, C19, C20, C21, C22, C23, C24: footprint Capacitors_SMD:C_1206_HandSoldering -> Capacitor_SMD:C_1206_3216Metric_Pad1.42x1.75mm_HandSolder; symbol C_Small -> Device1:C_Small
- D5: footprint LEDs:LED_1206 -> LED_SMD:LED_1206_3216Metric_Pad1.42x1.75mm_HandSolder; symbol Led_Small -> atari23MTS_Upgrade-rescue:Led_Small
- R10, R11, R12, R13, R14, R15, R16: footprint Resistors_SMD:R_1206_HandSoldering -> Resistor_SMD:R_1206_3216Metric_Pad1.42x1.75mm_HandSolder; symbol R_Small -> Device1:R_Small
- U14: footprint Housings_QFP:TQFP-100_14x14mm_Pitch0.5mm -> Package_QFP:TQFP-100-1EP_14x14mm_P0.5mm_EP5x5mm; symbol STM32F407VGTx -> MCU_ST_STM32F41:STM32F407VGTx
- XT2: symbol Crystal_Small -> Device1:Crystal_Small
