File: expansionslotspt.sch (KiCad schematic (older format))
At the start: 14 parts, among them J1 Conn_01x02, J2 Conn_01x02, J3 Conn_01x02, J4 Conn_01x02, J5 Conn_01x02, J6 Conn_01x02, J7 Conn_01x02, J8 Conn_01x02, U10 74LVC2G32, U11 74LVC2G08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

Commit message: Modified for dual processors board
Parts:
- removed J1, J2, J3, J4, J5, J6, J7, J8: Conn_01x02, Pin_Headers:Pin_Header_Straight_1x02, symbol Conn_01x02
- added P10, P11, P12, P13, P14, P7, P8, P9: CONN_01X02, Pin_Headers:Pin_Header_Straight_1x02, symbol CONN_01X02
Connections:
- net labels added: mB5, nRESET_MEM, ~mB5
- net labels removed: nRESET
- wire segments 59 -> 54
- no-connect marks 6 -> 5
Other:
- note added: "PBI Device Selection for UART/SPI Devices"
- note added: "RAM CHIP SELECT 0-1"
- note added: "This expansion can have a PBI device driver in ROM. It can be a RS232 (850 R: Interface compatible) or a GPIO 16 Channels Interface"
- moved on the sheet: U10A, U11A, U11B, U12, U9A, U9B

Commit message: C64 Emulation. First run on my beloved ATARI 130XE.
Parts:
- CART2: symbol ATARICARTRIDGE -> AmigaComponents:ATARICARTRIDGE
- ECI2: symbol ECIBUS -> AmigaComponents:ECIBUS
- P10, P11, P12, P13, P14, P7, P8, P9: footprint Pin_Headers:Pin_Header_Straight_1x02 -> Connector_PinHeader_2.54mm:PinHeader_1x02_P2.54mm_Vertical; symbol CONN_01X02 -> atari23MTS_Upgrade-rescue:CONN_01X02
- U10: footprint Housings_SSOP:TSSOP-8_3x3mm_Pitch0.65mm -> Package_SO:TSSOP-8_3x3mm_P0.65mm; symbol 74LVC2G32 -> 74xGxx1:74LVC2G32
- U11: footprint Housings_SSOP:TSSOP-8_3x3mm_Pitch0.65mm -> Package_SO:TSSOP-8_3x3mm_P0.65mm; symbol 74LVC2G08 -> 74xGxx1:74LVC2G08
- U12: footprint Housings_SSOP:TSSOP-8_3x3mm_Pitch0.65mm -> Package_SO:TSSOP-8_3x3mm_P0.65mm; symbol 74LVC2G74 -> 74xGxx1:74LVC2G74
- U9: footprint Housings_SSOP:SSOP-14_5.3x6.2mm_Pitch0.65mm -> Package_SO:SSOP-14_5.3x6.2mm_P0.65mm; symbol 74HCT04 -> 74xx1:74HCT04

Commit message: RetroBitLab library
Parts:
- CART2: symbol AmigaComponents:ATARICARTRIDGE -> RetroBitLab:ATARICARTRIDGE
- ECI2: symbol AmigaComponents:ECIBUS -> RetroBitLab:ECIBUS
Changed lines of the file:
@@
 $EndDescr
 $Comp
-L AmigaComponents:ATARICARTRIDGE CART2
+L RetroBitLab:ATARICARTRIDGE CART2
 U 1 1 5C2FF23F
 P 1850 2200
@@
 $EndComp
 $Comp
-L AmigaComponents:ECIBUS ECI2
+L RetroBitLab:ECIBUS ECI2
 U 1 1 5C2FF2C0
 P 4950 2250
