File: mcu.sch (KiCad schematic (older format))
At the start: 26 parts, among them J9 Micro_SD_Card_Det, U13 STM32F407VGTx

Commit message: Modified for dual processors board
Parts:
- removed D5: LED.AMBER, LEDs:LED_1206, symbol Led_Small
- removed R10, R9: 10k, Resistors_SMD:R_1206_HandSoldering, symbol R_Small
- removed R11, R12: 10K, Resistors_SMD:R_1206_HandSoldering, symbol R_Small
- removed R15: 220, Resistors_SMD:R_1206_HandSoldering, symbol R_Small
- XT1: footprint Crystal:Crystal_SMD_0603-4Pin_6.0x3.5mm_HandSoldering -> Crystals:Crystal_HC49-U_Vertical
Connections:
- net BOOT0 renamed BOOT0_CART
- net LEDAMBER: no longer names the net of U13.89 (PB3)
- net SWDCLK renamed SWDCLK_CART
- net SWDIO renamed SWDIO_CART
- net TP1: no longer names the net of U13.18 (PC3)
- net UART_RX_TTL: no longer names the net of U13.69 (PA10)
- net UART_TX_TTL: no longer names the net of U13.68 (PA9)
- net mPBISEL: no longer names the net of U13.7 (PC13)
- net mSPARE1: no longer names the net of U13.8 (PC14)
- net mSPARE2: no longer names the net of U13.9 (PC15)
- net mxA14: no longer names the net of U13.63 (PC6)
- net mxA15: no longer names the net of U13.64 (PC7)
- net mxA16: no longer names the net of U13.65 (PC8)
- net mxA17: no longer names the net of U13.66 (PC9)
- net mxA18: no longer names the net of U13.78 (PC10)
- net nRESET renamed nRESET_CART
- net ~mCHIP0: no longer names the net of U13.79 (PC11)
- net ~mCHIP1: no longer names the net of U13.80 (PC12)
- net ~mD1XX: no longer names the net of U13.91 (PB5)
- net ~mD8XX-DFXX: no longer names the net of U13.47 (PB10)
- net ~mEXSEL: no longer names the net of U13.92 (PB6)
- net ~mHALT: no longer names the net of U13.93 (PB7)
- net ~mIRQ: no longer names the net of U13.48 (PB11)
- net ~mMPD: no longer names the net of U13.96 (PB9)
- net ~mREF: no longer names the net of U13.51 (PB12)
- net ~mRST: no longer names the net of U13.95 (PB8)
- no-connect marks 29 -> 51
Other:
- note removed: "AMBER LED (EXPANSION MEMORY ACCESS SRAM)"
